File: NF1/kicad/NF1-MCP-V04/NF1-MCP2210-v04.kicad_pcb (KiCad board)
At the start: 2 copper layers, 42.5 x 25 mm, 53 parts, among them CN1 USB-A, P1 TST, P2 TST, P3 TST, P4 TST, P5 TST, P6 TST, P7 TST, P8 TST, U1 BD9C301FJ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

Commit message: minor fixes
Routing:
- net GND: track 512.6 -> 526.1 mm, vias 75 -> 77
Changed lines of the file:
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@@
     (thickness 1.6)
     (drawings 6)
-    (tracks 788)
+    (tracks 806)
     (zones 0)
     (modules 53)
@@
   )
   (setup
-    (last_trace_width 0.762)
+    (last_trace_width 0.508)
     (user_trace_width 0.254)
     (user_trace_width 0.381)
@@
       (drillshape 0)
       (scaleselection 1)
-      (outputdirectory plots/))
+      (outputdirectory tmp/))
   )
   (net 0 "")
@@
   (segment (start 131.03348 96.70364) (end 131.03348 95.8698) (width 0.762) (layer F.Cu) (net 10))
   (segment (start 131.03348 95.8698) (end 131.88696 95.01632) (width 0.762) (layer F.Cu) (net 10))
+  (segment (start 133.9088 95.9358) (end 133.59812 96.24648) (width 0.508) (layer F.Cu) (net 11))
+  (segment (start 133.59812 95.84516) (end 133.9088 95.53448) (width 0.508) (layer F.Cu) (net 11))
+  (segment (start 133.59812 96.24648) (end 133.59812 95.84516) (width 0.508) (layer F.Cu) (net 11))
+  (segment (start 133.9088 95.9358) (end 134.366 95.4786) (width 0.508) (layer F.Cu) (net 11))
+  (segment (start 134.366 93.5482) (end 134.1374 93.5482) (width 0.508) (layer F.Cu) (net 11))
+  (segment (start 134.874 93.0402) (end 134.366 93.5482) (width 0.508) (layer F.Cu) (net 11))
+  (segment (start 133.9088 93.7768) (end 133.9088 95.53448) (width 0.508) (layer F.Cu) (net 11))
+  (segment (start 134.1374 93.5482) (end 133.9088 93.7768) (width 0.508) (layer F.Cu) (net 11))
+  (segment (start 134.366 95.4786) (end 134.366 93.9292) (width 0.508) (layer F.Cu) (net 11))
+  (segment (start 127.16764 94.8944) (end 127.16764 94.17304) (width 0.508) (layer F.Cu) (net 11))
+  (segment (start 128.397 95.4024) (end 128.4478 95.4024) (width 0.508) (layer B.Cu) (net 11))
+  (segment (start 126.7206 93.726) (end 128.397 95.4024) (width 0.508) (layer B.Cu) (net 11))
+  (via (at 126.7206 93.726) (size 0.762) (layers F.Cu B.Cu) (net 11))
+  (segment (start 127.16764 94.17304) (end 126.7206 93.726) (width 0.508) (layer F.Cu) (net 11))
+  (segment (start 123.71942 96.21884) (end 121.67942 96.21884) (width 0.508) (layer F.Cu) (net 11))
+  (segment (start 121.67942 96.21884) (end 121.04442 96.85384) (width 0.508) (layer F.Cu) (net 11))
+  (via (at 128.7526 96.7994) (size 0.762) (layers F.Cu B.Cu) (net 11))
+  (segment (start 128.4478 96.4946) (end 128.7526 96.7994) (width 0.508) (layer B.Cu) (net 11))
+  (segment (start 128.4478 95.4024) (end 128.4478 96.4946) (width 0.508) (layer B.Cu) (net 11))
   (segment (start 121.54916 86.10346) (end 120.62714 86.10346) (width 0.762) (layer F.Cu) (net 11))
   (segment (start 120.65 89.3064) (end 120.65 89.9414) (width 0.762) (layer B.Cu) (net 11))
@@
   (segment (start 127.16764 96.40316) (end 127.16764 94.8944) (width 1.016) (layer F.Cu) (net 11))
   (segment (start 127.4826 96.71812) (end 128.07188 96.71812) (width 1.016) (layer F.Cu) (net 11))
-  (segment (start 128.15316 96.7994) (end 128.6256 96.7994) (width 1.016) (layer F.Cu) (net 11))
   (segment (start 128.07188 96.71812) (end 128.15316 96.7994) (width 1.016) (layer F.Cu) (net 11))
+  (segment (start 128.15316 96.7994) (end 128.7526 96.7994) (width 1.016) (layer F.Cu) (net 11))
+  (segment (start 128.7526 96.7994) (end 128.6256 96.7994) (width 1.016) (layer F.Cu) (net 11))
   (segment (start 127.16764 94.8944) (end 127.16764 94.98584) (width 1.016) (layer F.Cu) (net 11))
   (segment (start 127.16764 94.98584) (end 127.5842 95.4024) (width 1.016) (layer F.Cu) (net 11))
@@
   (segment (start 116.7892 89.9668) (end 115.1636 88.3412) (width 0.762) (layer B.Cu) (net 11))
   (segment (start 124.65304 93.0656) (end 124.65304 93.53296) (width 0.508) (layer F.Cu) (net 11))
+  (segment (start 124.65304 93.53296) (end 124.1044 94.0816) (width 0.508) (layer F.Cu) (net 11))
+  (segment (start 124.1044 94.0816) (end 122.0978 94.0816) (width 0.508) (layer F.Cu) (net 11))
+  (segment (start 122.0978 94.0816) (end 121.04442 95.13498) (width 0.508) (layer F.Cu) (net 11))
   (segment (start 121.04442 95.13498) (end 121.04442 96.85384) (width 0.508) (layer F.Cu) (net 11))
-  (segment (start 122.0978 94.0816) (end 121.04442 95.13498) (width 0.508) (layer F.Cu) (net 11))
-  (segment (start 124.1044 94.0816) (end 122.0978 94.0816) (width 0.508) (layer F.Cu) (net 11))
-  (segment (start 124.65304 93.53296) (end 124.1044 94.0816) (width 0.508) (layer F.Cu) (net 11))
   (segment (start 133.40842 93.1672) (end 133.40842 94.99854) (width 0.762) (layer F.Cu) (net 11))
   (segment (start 133.40842 94.99854) (end 133.39064 95.01632) (width 0.762) (layer F.Cu) (net 11))
@@
   (via (at 134.874 93.0402) (size 0.762) (layers F.Cu B.Cu) (net 11))
   (segment (start 134.8232 95.4024) (end 134.874 95.3516) (width 0.762) (layer B.Cu) (net 11))
+  (via (at 134.874 95.3516) (size 0.762) (layers F.Cu B.Cu) (net 11))
+  (segment (start 134.874 95.3516) (end 134.874 93.0402) (width 0.762) (layer F.Cu) (net 11))
   (segment (start 128.4478 95.4024) (end 134.8232 95.4024) (width 0.762) (layer B.Cu) (net 11))
-  (segment (start 134.874 95.3516) (end 134.874 93.0402) (width 0.762) (layer F.Cu) (net 11))
-  (via (at 134.874 95.3516) (size 0.762) (layers F.Cu B.Cu) (net 11))
   (segment (start 125.6157 96.7359) (end 125.1331 96.7359) (width 0.508) (layer F.Cu) (net 11))
   (segment (start 124.61604 96.21884) (end 123.71942 96.21884) (width 0.508) (layer F.Cu) (net 11))
@@
   (segment (start 128.4478 95.75292) (end 127.4826 96.71812) (width 0.762) (layer F.Cu) (net 11))
   (via (at 121.04442 96.85384) (size 0.762) (layers F.Cu B.Cu) (net 11))
-  (segment (start 127.16764 94.8944) (end 127.9398 94.8944) (width 0.762) (layer F.Cu) (net 11))
-  (segment (start 128.4478 95.4024) (end 127.9398 94.8944) (width 0.762) (layer F.Cu) (net 11))
   (via (at 128.4478 95.4024) (size 0.762) (layers F.Cu B.Cu) (net 11))
   (segment (start 122.49586 95.4024) (end 128.4478 95.4024) (width 0.762) (layer B.Cu) (net 11))
@@
     (polygon
       (pts
-        (xy 142.494 74.9808) (xy 142.4686 100.0506) (xy 142.4178 100.0252) (xy 119.1514 100.1014) (xy 119.15119 100.050566)
-        (xy 100.0252 100.0252) (xy 100.0252 75.057) (xy 114.7572 74.9046) (xy 114.760803 75.05692) (xy 142.494 74.9808)
+        (xy 142.5194 99.9998) (xy 142.0114 99.9744) (xy 135.509 100.1014) (xy 135.509 96.9264) (xy 132.0292 96.8756)
+        (xy 132.1054 100.0252) (xy 118.3132 100.076) (xy 118.315001 100.050567) (xy 100.0506 100.0252) (xy 99.9744 75.2856)
+        (xy 100.0252 75.0316) (xy 114.351513 74.955531) (xy 114.3508 74.8792) (xy 142.494 74.9808) (xy 142.5194 99.9998)
       )
     )
     (polygon
-      (pts        (xy 125.9586 80.9244) (xy 125.5776 78.0034) (xy 120.3706 77.7748) (xy 117.5004 80.4418) (xy 114.887182 80.399308)
-        (xy 115.0366 86.7156) (xy 119.1006 87.8586) (xy 119.101523 88.006381) (xy 119.1006 87.7824) (xy 125.1204 87.7824)
-        (xy 125.9586 80.9244)
+      (pts        (xy 126.5428 89.7128) (xy 126.238 81.7372) (xy 125.7046 79.8322) (xy 122.0216 79.6544) (xy 121.4882 80.264)
+        (xy 121.92 78.8416) (xy 119.5324 78.4098) (xy 117.5258 80.3656) (xy 115.7732 80.5434) (xy 115.2144 80.9752)
+        (xy 114.4016 80.3148) (xy 114.353686 75.18804) (xy 113.6904 82.042) (xy 113.2078 86.0298) (xy 113.2586 87.7316)
+        (xy 119.2276 87.7824) (xy 119.22011 87.885752) (xy 123.571 88.0618) (xy 126.5428 89.7128)
       )
     )
@@
     (polygon
       (pts
-        (xy 100.076 74.9808) (xy 142.5448 74.93) (xy 142.494 100.0252) (xy 100.076 100.0252) (xy 99.9744 75.3872)
+        (xy 100.076 74.93) (xy 142.5448 74.9808) (xy 142.494 100.1268) (xy 100.0252 100.076) (xy 100.076 75.2094)
       )
     )
