File: NF1/kicad/NF1-MCP-V05/NF1-MCP2210-v05.kicad_pcb (KiCad board)
At the start: 2 copper layers, 42.5 x 25 mm, 54 parts, among them CN1 USB-A, P1 TST, P2 TST, P3 TST, P4 TST, P5 TST, P6 TST, P7 TST, P8 TST, Q1 BSS138L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

Commit message: Add TechnoBit logo
Add TechnoBit logo for Marto74
Parts:
- added G***: LOGO, TechnoBit-LOGO, F.Cu at (112.3, 78.1)

Commit message: More tweaking with TechnoBit's logo
Parts:
- removed G***: LOGO, TechnoBit-LOGO
- added LOGO***: LOGO, TechnoBit-LOGO, F.Cu at (137.2, 77.1)
