File: NF1/kicad/NF1-MCP-V05/NF1-MCP2210-v05-TechnoBit.kicad_pcb (KiCad board)
At the start: 2 copper layers, 42.5 x 25 mm, 54 parts, among them CN1 USB-A, P1 TST, P2 TST, P3 TST, P4 TST, P5 TST, P6 TST, P7 TST, P8 TST, Q1 BSS138L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

Commit message: Add a separate copy for TechnoBit
update SCH version number and other minor tweaks
Parts:
- added LOGO***: LOGO, TechnoBit-LOGO, F.Cu at (137.2, 77.1)
Changed lines of the file:
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@@
     (tracks 776)
     (zones 0)
-    (modules 54)
+    (modules 55)
     (nets 30)
   )
@@
     )
   )
+  (module TechnoBit-LOGO (layer F.Cu)
+    (at 137.2108 77.1398)
+    (fp_text reference LOGO*** (at 0 2.286) (layer F.SilkS) hide
+      (effects (font (size 1.524 1.524) (thickness 0.3048)))
+    )
+    (fp_text value LOGO (at 0 -2.286) (layer F.SilkS) hide
+      (effects (font (size 1.524 1.524) (thickness 0.3048)))
+    )
+    (fp_poly (pts (xy 3.22326 1.09474) (xy 3.13436 1.23444) (xy 2.89306 1.3335) (xy 2.49682 1.397)
+      (xy 2.04978 1.42494) (xy 1.62814 1.4351) (xy 1.36144 1.42748) (xy 1.2319 1.39954)
+      (xy 1.2192 1.36398) (xy 1.3335 1.30556) (xy 1.55194 1.27) (xy 1.6764 1.26492)
+      (xy 2.00406 1.24714) (xy 2.3368 1.2065) (xy 2.62636 1.14808) (xy 2.8194 1.08712)
+      (xy 2.86004 1.06172) (xy 2.84734 0.97536) (xy 2.73558 0.85344) (xy 2.5781 0.74168)
+      (xy 2.42824 0.67818) (xy 2.40284 0.67564) (xy 2.2987 0.74422) (xy 2.286 0.80264)
+      (xy 2.21742 0.9144) (xy 2.16662 0.9271) (xy 2.16662 -0.30734) (xy 2.15392 -0.47752)
+      (xy 2.06756 -0.54102) (xy 1.9558 -0.57658) (xy 1.8923 -0.5461) (xy 1.85166 -0.41656)
+      (xy 1.81102 -0.18796) (xy 1.78562 0.03556) (xy 1.80848 0.1397) (xy 1.89738 0.16764)
+      (xy 1.93548 0.16764) (xy 2.08534 0.11176) (xy 2.11582 0.02032) (xy 2.13868 -0.18796)
+      (xy 2.16662 -0.30734) (xy 2.16662 0.9271) (xy 2.159 0.92964) (xy 2.05486 0.85598)
+      (xy 2.032 0.71882) (xy 1.98628 0.54864) (xy 1.905 0.508) (xy 1.80086 0.57658)
+      (xy 1.778 0.67564) (xy 1.72466 0.8128) (xy 1.651 0.84582) (xy 1.53924 0.77724)
+      (xy 1.524 0.70612) (xy 1.4605 0.5461) (xy 1.38176 0.46482) (xy 1.30556 0.34798)
+      (xy 1.29794 0.21336) (xy 1.34874 0.11938) (xy 1.43764 0.12446) (xy 1.49098 0.08382)
+      (xy 1.51892 -0.10668) (xy 1.524 -0.25146) (xy 1.50622 -0.52578) (xy 1.45796 -0.65786)
+      (xy 1.40462 -0.67818) (xy 1.27508 -0.74676) (xy 1.23444 -0.8128) (xy 1.19126 -0.96266)
+      (xy 1.2446 -1.01346) (xy 1.35382 -1.016) (xy 1.49606 -1.07696) (xy 1.524 -1.18618)
+      (xy 1.58242 -1.32842) (xy 1.69164 -1.35636) (xy 1.82626 -1.30302) (xy 1.86182 -1.15316)
+      (xy 1.92532 -0.96774) (xy 2.032 -0.90678) (xy 2.1463 -0.90424) (xy 2.21234 -1.00076)
+      (xy 2.25298 -1.19888) (xy 2.31648 -1.42494) (xy 2.39014 -1.4986) (xy 2.4511 -1.4224)
+      (xy 2.47396 -1.20904) (xy 2.46888 -1.11506) (xy 2.47142 -0.889) (xy 2.51206 -0.77216)
+      (xy 2.52984 -0.762) (xy 2.67208 -0.70104) (xy 2.86004 -0.55118) (xy 3.04546 -0.36068)
+      (xy 3.18008 -0.18034) (xy 3.21564 -0.07874) (xy 3.15214 0.07366) (xy 2.9972 0.2413)
+      (xy 2.97434 0.25654) (xy 2.82956 0.36322) (xy 2.82956 -0.14478) (xy 2.74066 -0.25654)
+      (xy 2.69494 -0.28702) (xy 2.55524 -0.381) (xy 2.48666 -0.37338) (xy 2.44348 -0.23876)
+      (xy 2.42316 -0.14986) (xy 2.40284 0.02032) (xy 2.46888 0.07874) (xy 2.5273 0.08382)
+      (xy 2.71526 0.0254) (xy 2.78638 -0.03556) (xy 2.82956 -0.14478) (xy 2.82956 0.36322)
+      (xy 2.73304 0.43434) (xy 2.97434 0.67564) (xy 3.16992 0.91186) (xy 3.22326 1.09474)
+      (xy 3.22326 1.09474)) (layer F.SilkS) (width 0.00254))
+    (fp_poly (pts (xy -2.71018 1.08966) (xy -2.78638 1.18618) (xy -2.98196 1.25222) (xy -3.16992 1.27)
+      (xy -3.28422 1.25476) (xy -3.33502 1.18364) (xy -3.33756 1.00838) (xy -3.32486 0.8636)
+      (xy -3.30708 0.61976) (xy -3.32994 0.50038) (xy -3.4163 0.45212) (xy -3.5052 0.44196)
+      (xy -3.63728 0.44196) (xy -3.70078 0.50038) (xy -3.72364 0.65786) (xy -3.72618 0.84582)
+      (xy -3.74142 1.08712) (xy -3.78206 1.23952) (xy -3.81 1.27) (xy -3.8608 1.1938)
+      (xy -3.89128 0.99822) (xy -3.89636 0.84582) (xy -3.9116 0.56642) (xy -3.95986 0.43942)
+      (xy -4.05384 0.4572) (xy -4.13258 0.52324) (xy -4.2164 0.57404) (xy -4.23418 0.48768)
+      (xy -4.1783 0.35814) (xy -3.99542 0.28448) (xy -3.6703 0.25908) (xy -3.55346 0.25908)
+      (xy -3.15468 0.28194) (xy -2.8702 0.32766) (xy -2.72542 0.39624) (xy -2.71018 0.42926)
+      (xy -2.77876 0.47244) (xy -2.921 0.4572) (xy -3.08356 0.44196) (xy -3.13436 0.52578)
+      (xy -3.13436 0.54102) (xy -3.07086 0.65786) (xy -3.00736 0.67564) (xy -2.89306 0.72136)
+      (xy -2.88036 0.762) (xy -2.94894 0.83566) (xy -3.00736 0.84582) (xy -3.11658 0.9144)
+      (xy -3.13436 0.98044) (xy -3.09372 1.07442) (xy -2.94386 1.06934) (xy -2.92354 1.06426)
+      (xy -2.76606 1.05156) (xy -2.71018 1.08966) (xy -2.71018 1.08966)) (layer F.SilkS) (width 0.00254))
+    (fp_poly (pts (xy -1.88722 1.12776) (xy -1.88976 1.13792) (xy -1.99136 1.21666) (xy -2.1844 1.24968)
+      (xy -2.3876 1.23444) (xy -2.51968 1.17094) (xy -2.59588 1.016) (xy -2.62636 0.8001)
+      (xy -2.57048 0.54356) (xy -2.43078 0.35814) (xy -2.24536 0.26416) (xy -2.05486 0.28956)
+      (xy -1.9558 0.37084) (xy -1.91516 0.44958) (xy -1.99898 0.48006) (xy -2.13614 0.47752)
+      (xy -2.31648 0.4826) (xy -2.40284 0.54864) (xy -2.43586 0.72644) (xy -2.44094 0.79248)
+      (xy -2.46888 1.12014) (xy -2.16408 1.08458) (xy -1.95834 1.0795) (xy -1.88722 1.12776)
+      (xy -1.88722 1.12776)) (layer F.SilkS) (width 0.00254))
+    (fp_poly (pts (xy -1.016 0.71374) (xy -1.03124 0.97028) (xy -1.0668 1.14046) (xy -1.10236 1.18364)
+      (xy -1.17094 1.11252) (xy -1.18618 1.016) (xy -1.23698 0.88138) (xy -1.39192 0.84582)
+      (xy -1.55702 0.889) (xy -1.62306 1.04394) (xy -1.6256 1.06426) (xy -1.6637 1.20396)
+      (xy -1.7145 1.2192) (xy -1.76022 1.08966) (xy -1.778 0.86614) (xy -1.76276 0.62738)
+      (xy -1.7272 0.47244) (xy -1.64338 0.34798) (xy -1.57988 0.3683) (xy -1.58496 0.508)
+      (xy -1.5875 0.63246) (xy -1.4732 0.6731) (xy -1.40716 0.67564) (xy -1.23698 0.64008)
+      (xy -1.18618 0.51054) (xy -1.14808 0.35052) (xy -1.10236 0.29464) (xy -1.05156 0.33782)
+      (xy -1.02362 0.53086) (xy -1.016 0.71374) (xy -1.016 0.71374)) (layer F.SilkS) (width 0.00254))
+    (fp_poly (pts (xy -0.08636 0.74676) (xy -0.09906 1.03378) (xy -0.13462 1.2192) (xy -0.17272 1.27)
+      (xy -0.2667 1.20142) (xy -0.39624 1.03378) (xy -0.44704 0.95504) (xy -0.62992 0.64262)
+      (xy -0.68834 0.91694) (xy -0.7493 1.15824) (xy -0.8001 1.2319) (xy -0.83566 1.13792)
+      (xy -0.84582 0.88138) (xy -0.82804 0.5334) (xy -0.77724 0.35306) (xy -0.68834 0.33528)
+      (xy -0.56642 0.4826) (xy -0.50038 0.59944) (xy -0.30734 0.97282) (xy -0.25146 0.65278)
+      (xy -0.19558 0.39116) (xy -0.14478 0.29464) (xy -0.10922 0.36322) (xy -0.0889 0.59436)
+      (xy -0.08636 0.74676) (xy -0.08636 0.74676)) (layer F.SilkS) (width 0.00254))
+    (fp_poly (pts (xy 0.8382 0.75438) (xy 0.83312 0.99568) (xy 0.74422 1.16586) (xy 0.635 1.21666)
+      (xy 0.635 0.762) (xy 0.61722 0.56134) (xy 0.5461 0.47752) (xy 0.42164 0.46482)
+      (xy 0.24892 0.51054) (xy 0.18288 0.6604) (xy 0.18796 0.92964) (xy 0.29464 1.06934)
+      (xy 0.44196 1.08458) (xy 0.57404 1.03378) (xy 0.62738 0.89916) (xy 0.635 0.762)
+      (xy 0.635 1.21666) (xy 0.55626 1.2573) (xy 0.32766 1.2573) (xy 0.13716 1.1684)
+      (xy 0.08636 1.1049) (xy 0.01016 0.83312) (xy 0.04572 0.56896) (xy 0.17526 0.36068)
+      (xy 0.381 0.25654) (xy 0.43688 0.254) (xy 0.6223 0.32766) (xy 0.762 0.51308)
+      (xy 0.8382 0.75438) (xy 0.8382 0.75438)) (layer F.SilkS) (width 0.00254))
+    (fp_poly (pts (xy 3.80492 0.82296) (xy 3.76682 1.01092) (xy 3.72364 1.09982) (xy 3.6703 1.143)
+      (xy 3.6449 1.0414) (xy 3.63982 0.90932) (xy 3.66014 0.70358) (xy 3.7084 0.5969)
+      (xy 3.72364 0.59182) (xy 3.78968 0.6604) (xy 3.80492 0.82296) (xy 3.80492 0.82296)) (layer F.SilkS) (width 0.00254))
+    (fp_poly (pts (xy 4.36626 1.05664) (xy 4.35864 1.09982) (xy 4.2418 1.1811) (xy 4.09956 1.09728)
+      (xy 4.08432 1.0795) (xy 3.95986 0.85852) (xy 3.93954 0.66802) (xy 4.03098 0.55626)
+      (xy 4.19862 0.55626) (xy 4.2672 0.59944) (xy 4.31038 0.69596) (xy 4.2545 0.7366)
+      (xy 4.15798 0.83058) (xy 4.16814 0.9525) (xy 4.27228 1.01346) (xy 4.2799 1.016)
+      (xy 4.36626 1.05664) (xy 4.36626 1.05664)) (layer F.SilkS) (width 0.00254))
+    (fp_poly (pts (xy 3.81 0.42164) (xy 3.74396 0.50546) (xy 3.72364 0.508) (xy 3.64236 0.44196)
+      (xy 3.63982 0.42164) (xy 3.70332 0.34036) (xy 3.72364 0.33782) (xy 3.80746 0.40132)
+      (xy 3.81 0.42164) (xy 3.81 0.42164)) (layer F.SilkS) (width 0.00254))
+  )
   (gr_text "NF1\nV0.5" (at 139.4841 96.9391) (layer F.Cu)
     (effects (font (size 1.016 1.016) (thickness 0.254)))
   )
-  (gr_text NanoFury (at 137.0457 77.0001) (layer F.SilkS)
+  (gr_text NanoFury (at 105.3465 85.1535 90) (layer F.SilkS)
     (effects (font (size 1.016 1.016) (thickness 0.2032)))
   )
-  (gr_text "NF1\nv0.5" (at 103.3526 76.4413) (layer F.SilkS)
+  (gr_text "NF1\nv0.5" (at 103.251 76.2) (layer F.SilkS)
     (effects (font (size 1.27 1.27) (thickness 0.254)))
   )
